Commit message: update model urdf file

File: GR1/GR1T1/urdf/GR1T1.urdf (robot description, URDF)
Before this commit: robot GR1T1, 33 links, 32 joints
Links:
- link l_foot_roll: geometry collision capsule length=0.24 radius=0.02; collision capsule length=0.24 radius=0.02
- link l_hand_pitch: geometry collision sphere radius=0.04; visual mesh filename=../meshes/l_hand_pitch.STL
- link l_hand_yaw: geometry collision capsule length=0.17 radius=0.035; visual mesh filename=../meshes/l_hand_yaw.STL
- link l_shank_pitch: geometry collision capsule length=0.2 radius=0.05; visual mesh filename=../meshes/l_shank_pitch.STL
- link l_thigh_pitch: geometry collision capsule length=0.25 radius=0.05; visual mesh filename=../meshes/l_thigh_pitch.STL
- link l_upper_arm_yaw: geometry collision capsule length=0.11 radius=0.03; visual mesh filename=../meshes/l_upper_arm_yaw.STL
- link r_foot_roll: geometry collision capsule length=0.24 radius=0.02; collision capsule length=0.24 radius=0.02
- link r_hand_pitch: geometry collision sphere radius=0.04; visual mesh filename=../meshes/r_hand_pitch.STL
- link r_hand_yaw: geometry collision capsule length=0.17 radius=0.035; visual mesh filename=../meshes/r_hand_yaw.STL
- link r_shank_pitch: geometry collision capsule length=0.2 radius=0.05; visual mesh filename=../meshes/r_shank_pitch.STL
- link r_thigh_pitch: geometry collision capsule length=0.25 radius=0.05; visual mesh filename=../meshes/r_thigh_pitch.STL
- link r_upper_arm_yaw: geometry collision capsule length=0.11 radius=0.03; visual mesh filename=../meshes/r_upper_arm_yaw.STL
- link waist_roll: geometry collision capsule length=0.1 radius=0.1; visual mesh filename=../meshes/waist_roll.STL
- link waist_yaw: geometry collision capsule length=0.05 radius=0.05; visual mesh filename=../meshes/waist_yaw.STL

File: GR1/GR1T2/urdf/GR1T2.urdf (robot description, URDF)
Before this commit: robot GR1T2, 35 links, 34 joints
Links:
- link l_foot_roll: geometry collision capsule length=0.24 radius=0.02; collision capsule length=0.24 radius=0.02
- link l_hand_pitch: geometry collision sphere radius=0.04; visual mesh filename=../meshes/Larm7.STL
- link l_hand_yaw: geometry collision capsule length=0.17 radius=0.035; visual mesh filename=../meshes/Larm5.STL
- link l_shank_pitch: geometry collision capsule length=0.2 radius=0.05; visual mesh filename=../meshes/Lleg4.STL
- link l_thigh_pitch: geometry collision capsule length=0.25 radius=0.05; visual mesh filename=../meshes/Lleg3.STL
- link l_upper_arm_yaw: geometry collision capsule length=0.11 radius=0.03; visual mesh filename=../meshes/Larm3.STL
- link link_waist_roll: geometry collision capsule length=0.1 radius=0.1; visual mesh filename=../meshes/waist1.STL
- link link_waist_yaw: geometry collision capsule length=0.05 radius=0.05; visual mesh filename=../meshes/waist3.STL
- link r_foot_roll: geometry collision capsule length=0.24 radius=0.02; collision capsule length=0.24 radius=0.02
- link r_hand_pitch: geometry collision sphere radius=0.04; visual mesh filename=../meshes/Rarm7.STL
- link r_hand_yaw: geometry collision capsule length=0.17 radius=0.035; visual mesh filename=../meshes/Rarm5.STL
- link r_shank_pitch: geometry collision capsule length=0.2 radius=0.05; visual mesh filename=../meshes/Rleg4.STL
- link r_thigh_pitch: geometry collision capsule length=0.25 radius=0.05; visual mesh filename=../meshes/Rleg3.STL
- link r_upper_arm_yaw: geometry collision capsule length=0.11 radius=0.03; visual mesh filename=../meshes/Rarm3.STL
