Commit message: [bug]added mass of screw into hand_yaw

File: GRX/GR1/GR1T1/URDF/urdf/GR1T1_fourier_hand.urdf (robot description, URDF)
Before this commit: robot GR1T1_simple_coll, 71 links, 70 joints
Links:
- link left_hand_yaw_link: mass 0.73 -> 0.89
- link right_hand_yaw_link: mass 0.73 -> 0.89

File: GRX/GR1/GR1T1/URDF/urdf/GR1T1_inspire_hand.urdf (robot description, URDF)
Before this commit: robot GR1T1_inspire_hand_simple_coll, 73 links, 72 joints
Links:
- link left_hand_yaw_link: mass 0.73 -> 0.89
- link right_hand_yaw_link: mass 0.73 -> 0.89

File: GRX/GR1/GR1T1/URDF/urdf/GR1T1_jaw.urdf (robot description, URDF)
Before this commit: robot GR1T1_jaw_simple_coll, 37 links, 36 joints
Links:
- link left_hand_yaw_link: mass 0.73 -> 0.89
- link right_hand_yaw_link: mass 0.73 -> 0.89

Commit message: [bug]fixed name error in urdf in left wrist roll joint, it was left wrist roll link

File: GRX/GR1/GR1T1/URDF/urdf/GR1T1_fourier_hand.urdf (robot description, URDF)
Before this commit: robot GR1T1_simple_coll, 71 links, 70 joints
Joints:
- removed joint left_wrist_roll_link
- added joint left_wrist_roll_joint: type revolute, parent left_hand_yaw_link, child left_hand_roll_link, origin xyz=0 0 -0.18765 rpy=0 0 0, axis 1 0 0, limit lower=-0.61 upper=0.61 effort=3.95 velocity=27.96

File: GRX/GR1/GR1T1/URDF/urdf/GR1T1_inspire_hand.urdf (robot description, URDF)
Before this commit: robot GR1T1_inspire_hand_simple_coll, 73 links, 72 joints
Joints:
- removed joint left_wrist_roll_link
- added joint left_wrist_roll_joint: type revolute, parent left_hand_yaw_link, child left_hand_roll_link, origin xyz=0 0 -0.18765 rpy=0 0 0, axis 1 0 0, limit lower=-0.61 upper=0.61 effort=3.95 velocity=27.96

File: GRX/GR1/GR1T1/URDF/urdf/GR1T1_jaw.urdf (robot description, URDF)
Before this commit: robot GR1T1_jaw_simple_coll, 37 links, 36 joints
Joints:
- removed joint left_wrist_roll_link
- added joint left_wrist_roll_joint: type revolute, parent left_hand_yaw_link, child left_hand_roll_link, origin xyz=0 0 -0.18765 rpy=0 0 0, axis 1 0 0, limit lower=-0.61 upper=0.61 effort=3.95 velocity=27.96
