Commit message: `GR1T1_jaw` and `GR1T2_jaw` urdf has been updated to added a `end_effecotr_link` aims to align with other urdf

File: GRX/GR1/GR1T1/URDF/urdf/GR1T1_jaw.urdf (robot description, URDF)
Before this commit: robot GR1T1_jaw_simple_coll, 37 links, 36 joints
Links:
- added link left_end_effector_link
- added link right_end_effector_link
Joints:
- added joint left_end_effector_joint: type fixed, parent left_hand_pitch_link, child left_end_effector_link, origin xyz=0 0 0 rpy=0 0 0
- added joint right_end_effector_joint: type fixed, parent right_hand_pitch_link, child right_end_effector_link, origin xyz=0 0 0 rpy=0 0 0
- joint left_jaw_joint: parent left_hand_pitch_link -> left_end_effector_link
- joint right_jaw_joint: parent right_hand_pitch_link -> right_end_effector_link

File: GRX/GR1/GR1T2/URDF/urdf/GR1T2_jaw.urdf (robot description, URDF)
Before this commit: robot GR1T2_jaw, 37 links, 36 joints
Links:
- added link left_end_effector_link
- added link right_end_effector_link
Joints:
- added joint left_end_effector_joint: type fixed, parent left_hand_pitch_link, child left_end_effector_link, origin xyz=0 0 0 rpy=0 0 0
- added joint right_end_effector_joint: type fixed, parent right_hand_pitch_link, child right_end_effector_link, origin xyz=0 0 0 rpy=0 0 0
- joint left_jaw_joint: parent left_hand_pitch_link -> left_end_effector_link
- joint right_jaw_joint: parent right_hand_pitch_link -> right_end_effector_link
