Commit message: 🐛 Fiexed the inertia for all GR1T2 related urdf

File: GRX/GR1/GR1T2/urdf/GR1T2_fourier_hand_6dof.urdf (robot description, URDF)
Before this commit: robot GR1T2_fourier_hand_6dof, 71 links, 70 joints
Links:
- link left_foot_pitch_link: mass 1.13 -> 0.057
- link left_foot_roll_link: mass 1.13 -> 1.07
- link left_hand_pitch_link: mass 0.055 -> 0.05
- link left_hand_roll_link: mass 0.055 -> 0.005
- link right_foot_pitch_link: mass 1.13 -> 0.057
- link right_foot_roll_link: mass 1.13 -> 1.07
- link right_hand_pitch_link: mass 0.055 -> 0.05
- link right_hand_roll_link: mass 0.055 -> 0.005

File: GRX/GR1/GR1T2/urdf/GR1T2_inspire_hand.urdf (robot description, URDF)
Before this commit: robot GR1T2_inspire_hand, 73 links, 72 joints
Links:
- link left_foot_pitch_link: mass 1.13 -> 0.057
- link left_foot_roll_link: mass 1.13 -> 1.07
- link left_hand_pitch_link: mass 0.055 -> 0.05
- link left_hand_roll_link: mass 0.055 -> 0.005
- link right_foot_pitch_link: mass 1.13 -> 0.057
- link right_foot_roll_link: mass 1.13 -> 1.07
- link right_hand_pitch_link: mass 0.055 -> 0.05
- link right_hand_roll_link: mass 0.055 -> 0.005

File: GRX/GR1/GR1T2/urdf/GR1T2_jaw.urdf (robot description, URDF)
Before this commit: robot GR1T2_jaw, 39 links, 38 joints
Links:
- link left_foot_pitch_link: mass 1.13 -> 0.057
- link left_foot_roll_link: mass 1.13 -> 1.07
- link left_hand_roll_link: mass 0.055 -> 0.005
- link right_foot_pitch_link: mass 1.13 -> 0.057
- link right_foot_roll_link: mass 1.13 -> 1.07
- link right_hand_roll_link: mass 0.055 -> 0.005

File: GRX/GR1/GR1T2/urdf/GR1T2_nohand.urdf (robot description, URDF)
Before this commit: robot GR1T2_nohand, 37 links, 36 joints
Links:
- link left_foot_pitch_link: mass 1.13 -> 0.057
- link left_foot_roll_link: mass 1.13 -> 1.07
- link left_hand_pitch_link: mass 0.055 -> 0.05
- link left_hand_roll_link: mass 0.055 -> 0.005
- link right_foot_pitch_link: mass 1.13 -> 0.057
- link right_foot_roll_link: mass 1.13 -> 1.07
- link right_hand_pitch_link: mass 0.055 -> 0.05
- link right_hand_roll_link: mass 0.055 -> 0.005
