Commit message: ✨ GR2v3.0.1 has been released 🎨 GR2 foot has been renamed to  GR2v2.1.1

File: GRX/GR2/GR2v3.0.1/urdf/GR2v3.0.1.urdf (robot description, URDF)
Before this commit: robot GR2_foot, 35 links, 34 joints
Links:
- link base_link: mass 6.36 -> 6.6598; geometry collision box size=0.18 0.06 0.02; collision box size=0.18 0.06 0.02
- link camera_link: mass 0.07 -> 0; geometry 
- link head_pitch_link: mass 1.29 -> 1.6096; geometry collision sphere radius=0.09; visual mesh filename=../meshes/head_pitch_link.STL
- link head_yaw_link: mass 0.21 -> 0.1402
- link imu_link: geometry 
- link left_end_effector_link: mass 0.55 -> 0; geometry 
- link left_foot_pitch_link: mass 0.6548 -> 0.17877; geometry visual mesh filename=../meshes/left_foot_pitch_link.STL
- link left_foot_roll_link: mass 0.09 -> 1.1232; geometry collision cylinder length=0.28 radius=0.025; collision cylinder length=0.28 radius=0.025
- link left_hand_pitch_link: mass 0.46 -> 0.45716
- link left_hand_roll_link: mass 0.2 -> 0.20259
- link left_hand_yaw_link: mass 1.04 -> 1.0855; geometry collision cylinder length=0.115 radius=0.045; visual mesh filename=../meshes/left_hand_yaw_link.STL
- link left_lower_arm_pitch_link: mass 0.48 -> 0.45807
- link left_shank_pitch_link: mass 3.08 -> 3.5932; geometry collision cylinder length=0.18 radius=0.05; visual mesh filename=../meshes/left_shank_pitch_link.STL
- link left_thigh_pitch_link: mass 2.57 -> 2.61
- link left_thigh_roll_link: mass 1.34 -> 1.3487; geometry collision cylinder length=0.18 radius=0.05; visual mesh filename=../meshes/left_thigh_roll_link.STL
- link left_thigh_yaw_link: mass 5.04 -> 5.1152; geometry collision cylinder length=0.26 radius=0.06; visual mesh filename=../meshes/left_thigh_yaw_link.STL
- link left_upper_arm_pitch_link: mass 1.35 -> 1.3432
- link left_upper_arm_roll_link: mass 0.96 -> 0.96142; geometry collision sphere radius=0.045; visual mesh filename=../meshes/left_upper_arm_roll_link.STL
- link left_upper_arm_yaw_link: mass 1.32 -> 1.3181; geometry collision cylinder length=0.10 radius=0.04; visual mesh filename=../meshes/left_upper_arm_yaw_link.STL
- link right_end_effector_link: mass 0.55 -> 0; geometry 
- link right_foot_pitch_link: mass 0.6548 -> 0.17877; geometry visual mesh filename=../meshes/right_foot_pitch_link.STL
- link right_foot_roll_link: mass 0.09 -> 1.1232; geometry collision cylinder length=0.28 radius=0.025; collision cylinder length=0.28 radius=0.025
- link right_hand_pitch_link: mass 0.46 -> 0.45716
- link right_hand_roll_link: mass 0.2 -> 0.20259
- link right_hand_yaw_link: mass 1.04 -> 1.0855; geometry collision cylinder length=0.1155 radius=0.045; visual mesh filename=../meshes/right_hand_yaw_link.STL
- link right_lower_arm_pitch_link: mass 0.48 -> 0.45807
- link right_shank_pitch_link: mass 3.08 -> 3.5932; geometry collision cylinder length=0.18 radius=0.05; visual mesh filename=../meshes/right_shank_pitch_link.STL
- link right_thigh_pitch_link: mass 2.57 -> 2.61
- link right_thigh_roll_link: mass 1.34 -> 1.3487; geometry collision cylinder length=0.18 radius=0.05; visual mesh filename=../meshes/right_thigh_roll_link.STL
- link right_thigh_yaw_link: mass 5.04 -> 5.1152; geometry collision cylinder length=0.26 radius=0.06; visual mesh filename=../meshes/right_thigh_yaw_link.STL
- link right_upper_arm_pitch_link: mass 1.35 -> 1.3432
- link right_upper_arm_roll_link: mass 0.96 -> 0.96142; geometry collision sphere radius=0.045; visual mesh filename=../meshes/right_upper_arm_roll_link.STL
- link right_upper_arm_yaw_link: mass 1.32 -> 1.3181; geometry collision cylinder length=0.1 radius=0.040; visual mesh filename=../meshes/right_upper_arm_yaw_link.STL
- link torso_link: mass 14.97 -> 14.058; geometry collision cylinder length=0.3 radius=0.15; visual mesh filename=../meshes/torso_link.STL
- link waist_yaw_link: mass 0.69 -> 0.67252
Joints:
- joint camera_joint: origin xyz=0.090579 0 0.091065 rpy=0 0.12217 0 -> xyz=0.11296 0 0.09815 rpy=0 0 0
- joint head_pitch_joint: limit lower=-0.523 upper=0.663 effort=29.4 velocity=4.58 -> lower=-0.5236 upper=0.5236 effort=17.325 velocity=9.1627; origin xyz=0 0 0.07005 rpy=0 0 0 -> xyz=0 0 0.044185 rpy=0 0 0
- joint head_yaw_joint: limit lower=-1.396 upper=1.396 effort=29.4 velocity=4.58 -> lower=-1.3963 upper=1.3963 effort=17.325 velocity=9.1627; origin xyz=0.001 0 0.08575 rpy=0 0 0 -> xyz=0.001 0 0.11061 rpy=0 0 0
- joint left_ankle_pitch_joint: limit lower=-0.785 upper=0.785 effort=51 velocity=6.18 -> lower=-0.7854 upper=0.7854 effort=54.33 velocity=14.745; origin xyz=0 0 0 rpy=0 0 0 -> xyz=0 0 -0.406 rpy=0 0 0; parent left_foot_roll_link -> left_shank_pitch_link
- joint left_ankle_roll_joint: limit lower=-0.436 upper=0.436 effort=29.1 velocity=13.61 -> lower=-0.38397 upper=0.38397 effort=29.835 velocity=16.755; origin xyz=0 0 -0.406 rpy=0 0 0 -> xyz=0 0 0 rpy=0 0 0; parent left_shank_pitch_link -> left_foot_pitch_link
- joint left_elbow_pitch_joint: limit lower=-1.526 upper=0.479 effort=47.4 velocity=4.97 -> lower=-1.5272 upper=0.47997 effort=42.75 velocity=6.283; origin xyz=0 0 -0.13252 rpy=0 -0.3927 0 -> xyz=0 0 -0.16111 rpy=0 -0.3926 0
- joint left_end_effector_joint: origin xyz=0 0 -0.045 rpy=0 0 0 -> xyz=0 0 -0.052 rpy=0 0 0
- joint left_hip_pitch_joint: limit lower=-2.617 upper=2.617 effort=360 velocity=5.55 -> lower=-2.618 upper=2.618 effort=366.05 velocity=6.4997; origin xyz=0 0.05513 -0.111 rpy=-0.5236 0 0 -> xyz=0 0.076867 -0.12355 rpy=-0.5236 0 0
- joint left_hip_roll_joint: limit lower=-0.419 upper=1.57 effort=114 velocity=10.47 -> lower=-0.59341 upper=1.5708 effort=95.472 velocity=12.362; origin xyz=-0.0855 0.098 0 rpy=0.5236 0 0 -> xyz=-0.062 0.0729 0 rpy=0.5236 0 0
- joint left_hip_yaw_joint: limit lower=-0.698 upper=1.57 effort=51 velocity=6.18 -> lower=-0.69813 upper=1.5708 effort=54.33 velocity=14.745; origin xyz=0.0855 0 0 rpy=0 0 0 -> xyz=0.062 0 -0.03495 rpy=0 0 0
- joint left_knee_pitch_joint: limit lower=-0.087 upper=2.355 effort=360 velocity=5.55 -> lower=-0.087266 upper=2.3562 effort=366.05 velocity=6.4997; origin xyz=0 0 -0.378 rpy=0 0 0 -> xyz=0 0 -0.34305 rpy=0 0 0
- joint left_shoulder_pitch_joint: limit lower=-2.966 upper=1.919 effort=82.5 velocity=3.24 -> lower=-2.9671 upper=2.9671 effort=74.45 velocity=7.7568; origin xyz=0 0.128 0 rpy=0 0 0 -> xyz=0 0.15115 0 rpy=0 0 0
- joint left_shoulder_roll_joint: limit lower=-0.523 upper=2.791 effort=82.5 velocity=3.24 -> lower=-0.5236 upper=2.7925 effort=74.45 velocity=7.7568; origin xyz=0 0.102 0 rpy=0 0 0 -> xyz=0 0.078848 0 rpy=0 0 0
- joint left_shoulder_yaw_joint: limit lower=-1.832 upper=1.832 effort=47.4 velocity=4.97 -> lower=-1.8326 upper=1.8326 effort=42.75 velocity=6.283; origin xyz=0 0 -0.12298 rpy=0 0 0 -> xyz=0 0 -0.09438 rpy=0 0 0
- joint left_wrist_pitch_joint: limit lower=-0.611 upper=0.611 effort=29.4 velocity=4.58 -> lower=-0.61087 upper=0.61087 effort=17.325 velocity=9.1627; origin xyz=0 0 -0.13208 rpy=0 0 0 -> xyz=0 0 -0.16102 rpy=0 0 0
- joint left_wrist_roll_joint: limit lower=-0.959 upper=0.959 effort=29.4 velocity=4.58 -> lower=-0.95993 upper=0.95993 effort=17.325 velocity=9.1627
- joint left_wrist_yaw_joint: limit lower=-1.832 upper=1.832 effort=29.4 velocity=4.58 -> lower=-1.8326 upper=1.8326 effort=17.325 velocity=9.1627; origin xyz=0 0 -0.086418 rpy=0 0 0 -> xyz=0 0 -0.058525 rpy=0 0 0
- joint right_ankle_pitch_joint: limit lower=-0.785 upper=0.785 effort=51 velocity=6.18 -> lower=-0.7854 upper=0.7854 effort=54.33 velocity=14.745; origin xyz=0 0 0 rpy=0 0 0 -> xyz=0 0 -0.406 rpy=0 0 0; parent right_foot_roll_link -> right_shank_pitch_link
- joint right_ankle_roll_joint: limit lower=-0.436 upper=0.436 effort=29.1 velocity=13.61 -> lower=-0.38397 upper=0.38397 effort=29.835 velocity=16.755; origin xyz=0 0 -0.406 rpy=0 0 0 -> xyz=0 0 0 rpy=0 0 0; parent right_shank_pitch_link -> right_foot_pitch_link
- joint right_elbow_pitch_joint: limit lower=-1.526 upper=0.479 effort=47.4 velocity=4.97 -> lower=-1.5272 upper=0.47997 effort=42.75 velocity=6.283; origin xyz=0 0 -0.13252 rpy=0 -0.3927 0 -> xyz=0 0 -0.16111 rpy=0 -0.39265 0
- joint right_end_effector_joint: origin xyz=0 0 -0.045 rpy=0 0 0 -> xyz=0 0 -0.052 rpy=0 0 0
- joint right_hip_pitch_joint: limit lower=-2.617 upper=2.617 effort=360 velocity=5.55 -> lower=-2.618 upper=2.618 effort=366.05 velocity=6.4997; origin xyz=0 -0.05513 -0.111 rpy=0.5236 0 0 -> xyz=0 -0.076867 -0.12355 rpy=0.5236 0 0
- joint right_hip_roll_joint: limit lower=-1.57 upper=0.419 effort=114 velocity=10.47 -> lower=-1.5708 upper=0.59341 effort=95.472 velocity=12.362; origin xyz=-0.0855 -0.098 0 rpy=-0.5236 0 0 -> xyz=-0.062 -0.0729 0 rpy=-0.5236 0 0
- joint right_hip_yaw_joint: limit lower=-1.57 upper=0.698 effort=51 velocity=6.18 -> lower=-1.5708 upper=0.69813 effort=54.33 velocity=14.745; origin xyz=0.0855 0 0 rpy=0 0 0 -> xyz=0.062 0 -0.03495 rpy=0 0 0
- joint right_knee_pitch_joint: limit lower=-0.087 upper=2.355 effort=360 velocity=5.55 -> lower=-0.087266 upper=2.3562 effort=366.05 velocity=6.4997; origin xyz=0 0 -0.378 rpy=0 0 0 -> xyz=0 0 -0.34305 rpy=0 0 0
- joint right_shoulder_pitch_joint: limit lower=-2.966 upper=1.919 effort=82.5 velocity=3.24 -> lower=-2.9671 upper=2.9671 effort=74.45 velocity=7.7568; origin xyz=0 -0.128 0 rpy=0 0 0 -> xyz=0 -0.1585 0 rpy=0 0 0
- joint right_shoulder_roll_joint: limit lower=-2.791 upper=0.523 effort=82.5 velocity=3.24 -> lower=-2.7925 upper=0.5236 effort=74.45 velocity=7.7568; origin xyz=0 -0.102 0 rpy=0 0 0 -> xyz=0 -0.071498 0 rpy=0 0 0
- joint right_shoulder_yaw_joint: limit lower=-1.832 upper=1.832 effort=47.4 velocity=4.97 -> lower=-1.8326 upper=1.8326 effort=42.75 velocity=6.283; origin xyz=0 0 -0.12298 rpy=0 0 0 -> xyz=0 0 -0.09438 rpy=0 0 0
- joint right_wrist_pitch_joint: limit lower=-0.611 upper=0.611 effort=29.4 velocity=4.58 -> lower=-0.61087 upper=0.61087 effort=17.325 velocity=9.1627; origin xyz=0 0 -0.13208 rpy=0 0 0 -> xyz=0 0 -0.16102 rpy=0 0 0
- joint right_wrist_roll_joint: limit lower=-0.959 upper=0.959 effort=29.4 velocity=4.58 -> lower=-0.95993 upper=0.95993 effort=17.325 velocity=9.1627
- joint right_wrist_yaw_joint: limit lower=-1.832 upper=1.832 effort=29.4 velocity=4.58 -> lower=-1.8326 upper=1.8326 effort=17.325 velocity=9.1627; origin xyz=0 0 -0.086418 rpy=0 0 0 -> xyz=0 0 -0.058525 rpy=0 0 0
- joint torso_joint: origin xyz=0 0 0.4135 rpy=0 0 0 -> xyz=0 0 0.39681 rpy=0 0 0
- joint waist_yaw_joint: limit lower=-2.617 upper=2.617 effort=82.5 velocity=3.24 -> lower=-2.618 upper=2.618 effort=74.45 velocity=7.7568; origin xyz=0 0 -0.0335 rpy=0 0 0 -> xyz=0 0 -0.0159 rpy=0 0 0
