Commit message: ✨ fourier hand version updated. Also alone with gr1t1 and gr1t2

File: Dexterous_hand/fourier_hand_6dof/urdf/fourier_left_hand_6dof.urdf (robot description, URDF)
Before this commit: robot fourier_left_hand_6dof, 17 links, 16 joints
Links:
- removed link L_thumb_proximal_base_link
- removed link L_thumb_proximal_link
- added link L_thumb_proximal_pitch_link, mass 0.060766; collision mesh filename=../meshes/fourier_hand_6dof/L_thumb_proximal_pitch_link.STL; visual mesh filename=../meshes/fourier_hand_6dof/L_thumb_proximal_pitch_link.STL
- added link L_thumb_proximal_yaw_link, mass 0.0084328; collision mesh filename=../meshes/fourier_hand_6dof/L_thumb_proximal_yaw_link.STL; visual mesh filename=../meshes/fourier_hand_6dof/L_thumb_proximal_yaw_link.STL
- link L_hand_base_link: mass 0.306 -> 0.29928
- link L_index_intermediate_link: mass 0.01292544 -> 0.0027085
- link L_index_proximal_link: mass 0.019117 -> 0.011244
- link L_middle_intermediate_link: mass 0.01535007 -> 0.0032739
- link L_middle_proximal_link: mass 0.01911771 -> 0.011244
- link L_pinky_intermediate_link: mass 0.00568707 -> 0.0024076
- link L_pinky_proximal_link: mass 0.01911771 -> 0.011244
- link L_ring_intermediate_link: mass 0.01292544 -> 0.0027085
- link L_ring_proximal_link: mass 0.01911771 -> 0.011244
- link L_thumb_distal_link: mass 0.02031766 -> 0.018024
Joints:
- joint L_index_intermediate_joint: limit lower=-1.74 upper=0 effort=10 velocity=0.8 -> lower=-1.791 upper=0 effort=0 velocity=0; mimic joint=L_index_proximal_joint multiplier=1.128 offset=0 -> joint=L_index_proximal_joint multiplier=0.975 offset=0; origin xyz=0.031532 -0.0054551 0 rpy=0 0 -6.8256E-05 -> xyz=0.031533 -0.0054444 0 rpy=0 0.00014037 -0.0018338
- joint L_index_proximal_joint: limit lower=-1.57 upper=0 effort=10 velocity=0.8 -> lower=-1.602 upper=0 effort=0 velocity=0; origin xyz=0.026869 -0.012293 -0.095989 rpy=0.0013057 1.5184 0.0013039 -> xyz=0.026868 -0.0123 -0.093989 rpy=0 1.5184 0
- joint L_index_tip_joint: origin xyz=0.038 -0.0015 0 rpy=0 0 0 -> xyz=0.0390 -0.0020 0 rpy=0 0 0
- joint L_middle_intermediate_joint: limit lower=-1.74 upper=0 effort=10 velocity=0.8 -> lower=-1.791 upper=0 effort=0 velocity=0; mimic joint=L_middle_proximal_joint multiplier=1.131 offset=0 -> joint=L_middle_proximal_joint multiplier=0.975 offset=0; origin xyz=0.031662 -0.0046408 0 rpy=0 0 -6.835E-05 -> xyz=0.031521 -0.0055139 0 rpy=0 0.00015517 0.0048744
- joint L_middle_proximal_joint: limit lower=-1.57 upper=0 effort=10 velocity=0.8 -> lower=-1.603 upper=0 effort=0 velocity=0; origin xyz=0.0085012 -0.012293 -0.097993 rpy=1.394 1.5707 1.394 -> xyz=0.0085 -0.0123 -0.095992 rpy=0 1.5708 0
- joint L_middle_tip_joint: origin xyz=0.045 0.0005 0 rpy=0 0 0 -> xyz=0.047 -0.0025 0 rpy=0 0 0
- joint L_pinky_intermediate_joint: limit lower=-1.74 upper=0 effort=10 velocity=0.8 -> lower=-1.796 upper=0 effort=0 velocity=0; mimic joint=L_pinky_proximal_joint multiplier=1.129 offset=0 -> joint=L_pinky_proximal_joint multiplier=0.975 offset=0; origin xyz=0.031338 -0.0064763 0 rpy=0 0 -6.7976E-05 -> xyz=0.031532 -0.005451 0 rpy=0 0.00032164 -0.011403
- joint L_pinky_proximal_joint: limit lower=-1.57 upper=0 effort=10 velocity=0.8 -> lower=-1.602 upper=0 effort=0 velocity=0; origin xyz=-0.028227 -0.012293 -0.096013 rpy=3.1409 1.4661 3.1409 -> xyz=-0.028228 -0.0123 -0.094012 rpy=3.1416 1.4661 3.1416
- joint L_pinky_tip_joint: origin xyz=0.031 -0.0040 0 rpy=0 0 0 -> xyz=0.033 -0.0015 0 rpy=0 0 0
- joint L_ring_intermediate_joint: limit lower=-1.74 upper=0 effort=10 velocity=0.8 -> lower=-1.798 upper=0 effort=0 velocity=0; mimic joint=L_ring_proximal_joint multiplier=1.143 offset=0 -> joint=L_ring_proximal_joint multiplier=0.975 offset=0; origin xyz=0.031532 -0.0054551 0 rpy=0 0 -6.8256E-05 -> xyz=0.031531 -0.0054567 0.00025 rpy=0 0.00014037 -0.0025338
- joint L_ring_proximal_joint: limit lower=-1.57 upper=0 effort=10 velocity=0.8 -> lower=-1.602 upper=0 effort=0 velocity=0; origin xyz=-0.00996 -0.012293 -0.097938 rpy=3.1403 1.5184 3.1403 -> xyz=-0.010211 -0.0123 -0.095924 rpy=3.1416 1.5184 3.1416
- joint L_ring_tip_joint: origin xyz=0.038 -0.002 0 rpy=0 0 0 -> xyz=0.0385 -0.0015 0 rpy=0 0 0
- joint L_thumb_distal_joint: limit lower=0 upper=1.23 effort=10 velocity=0.8 -> lower=0 upper=1.267 effort=0 velocity=0; mimic joint=L_thumb_proximal_pitch_joint multiplier=0.974 offset=0 -> joint=L_thumb_proximal_pitch_joint multiplier=1.06 offset=0; origin xyz=0.061549 0.0074616 0 rpy=0 0 1.221E-05 -> xyz=0.061549 0.007464 0 rpy=0 1.7448E-05 -0.055652; parent L_thumb_proximal_link -> L_thumb_proximal_pitch_link
- joint L_thumb_proximal_pitch_joint: child L_thumb_proximal_link -> L_thumb_proximal_pitch_link; limit lower=0 upper=1.22 effort=10 velocity=0.8 -> lower=0 upper=1.159 effort=0 velocity=0; origin xyz=0.02175 0 0 rpy=-1.5707 0 0 -> xyz=0.021749 -0.00016321 0 rpy=-1.5708 0 -0.0052052; parent L_thumb_proximal_base_link -> L_thumb_proximal_yaw_link
- joint L_thumb_proximal_yaw_joint: child L_thumb_proximal_base_link -> L_thumb_proximal_yaw_link; limit lower=-1.74 upper=0 effort=10 velocity=0.8 -> lower=-1.676 upper=0 effort=0 velocity=0; origin xyz=0.022 -0.015498 -0.025093 rpy=0 -1.221E-05 0 -> xyz=0.022 -0.0155 -0.022992 rpy=0 0 0
- joint L_thumb_tip_joint: origin xyz=0.031 -0.001 0 rpy=0 0 0 -> xyz=0.0305 -0.001 0 rpy=0 0 0

File: Dexterous_hand/fourier_hand_6dof/urdf/fourier_right_hand_6dof.urdf (robot description, URDF)
Before this commit: robot fourier_right_hand_6dof, 17 links, 16 joints
Links:
- removed link R_thumb_proximal_base_link
- removed link R_thumb_proximal_link
- added link R_thumb_proximal_pitch_link, mass 0.060766; collision mesh filename=../meshes/fourier_hand_6dof/R_thumb_proximal_pitch_link.STL; visual mesh filename=../meshes/fourier_hand_6dof/R_thumb_proximal_pitch_link.STL
- added link R_thumb_proximal_yaw_link, mass 0.0084327; collision mesh filename=../meshes/fourier_hand_6dof/R_thumb_proximal_yaw_link.STL; visual mesh filename=../meshes/fourier_hand_6dof/R_thumb_proximal_yaw_link.STL
- link R_hand_base_link: mass 0.306 -> 0.2993
- link R_index_intermediate_link: mass 0.01292544 -> 0.0027085
- link R_index_proximal_link: mass 0.01911771 -> 0.011244
- link R_middle_intermediate_link: mass 0.01535 -> 0.0032739
- link R_middle_proximal_link: mass 0.01911771 -> 0.011244
- link R_pinky_intermediate_link: mass 0.00568707 -> 0.0024076
- link R_pinky_proximal_link: mass 0.01911771 -> 0.011244
- link R_ring_intermediate_link: mass 0.012925 -> 0.0027085
- link R_ring_proximal_link: mass 0.01911771 -> 0.011244
- link R_thumb_distal_link: mass 0.01974135 -> 0.018024
Joints:
- joint R_index_intermediate_joint: limit lower=-1.74 upper=0 effort=10 velocity=0.8 -> lower=-1.791 upper=0 effort=0 velocity=0; mimic joint=R_index_proximal_joint multiplier=1.128 offset=0 -> joint=R_index_proximal_joint multiplier=0.975 offset=0; origin xyz=0.031532 -0.0054551 0 rpy=0 0 0 -> xyz=0.031535 -0.0054349 0 rpy=0 0.00014037 -0.0012936
- joint R_index_proximal_joint: limit lower=-1.57 upper=0 effort=10 velocity=0.8 -> lower=-1.602 upper=0 effort=0 velocity=0; origin xyz=0.026864 0.012307 -0.095892 rpy=-3.1403 1.5184 0.0013039 -> xyz=0.026866 0.0123 -0.09399 rpy=3.1416 1.5184 0
- joint R_index_tip_joint: origin xyz=0.038 -0.0015 0 rpy=0 0 0 -> xyz=0.0390 -0.0020 0 rpy=0 0 0
- joint R_middle_intermediate_joint: limit lower=-1.74 upper=0 effort=10 velocity=0.8 -> lower=-1.791 upper=0 effort=0 velocity=0; mimic joint=R_middle_proximal_joint multiplier=1.131 offset=0 -> joint=R_middle_proximal_joint multiplier=0.975 offset=0; origin xyz=0.031662 -0.0046408 0 rpy=0 0 0 -> xyz=0.031531 -0.0054597 0 rpy=0 0.00015517 0.007959
- joint R_middle_proximal_joint: limit lower=-1.57 upper=0 effort=10 velocity=0.8 -> lower=-1.603 upper=0 effort=0 velocity=0; origin xyz=0.0084962 0.012307 -0.097896 rpy=-1.7476 1.5707 1.394 -> xyz=0.0085 0.0123 -0.096 rpy=3.1416 1.5708 0
- joint R_middle_tip_joint: origin xyz=0.045 0.0005 0 rpy=0 0 0 -> xyz=0.047 -0.0025 0 rpy=0 0 0
- joint R_pinky_intermediate_joint: limit lower=-1.74 upper=0 effort=10 velocity=0.8 -> lower=-1.796 upper=0 effort=0 velocity=0; mimic joint=R_pinky_proximal_joint multiplier=1.129 offset=0 -> joint=R_pinky_proximal_joint multiplier=0.975 offset=0; origin xyz=0.031338 -0.0064763 0 rpy=0 0 6.7976E-05 -> xyz=0.031474 -0.0057796 0 rpy=0 7.8504E-05 -0.030132
- joint R_pinky_proximal_joint: limit lower=-1.57 upper=0 effort=10 velocity=0.8 -> lower=-1.602 upper=0 effort=0 velocity=0; origin xyz=-0.028232 0.012307 -0.095916 rpy=-0.00065397 1.4661 3.1409 -> xyz=-0.028223 0.0123 -0.093963 rpy=0 1.4661 3.1416
- joint R_pinky_tip_joint: origin xyz=0.031 -0.004 0 rpy=0 0 0 -> xyz=0.033 -0.0015 0 rpy=0 0 0
- joint R_ring_intermediate_joint: limit lower=-1.74 upper=0 effort=10 velocity=0.8 -> lower=-1.798 upper=0 effort=0 velocity=0; mimic joint=R_ring_proximal_joint multiplier=1.143 offset=0 -> joint=R_ring_proximal_joint multiplier=0.975 offset=0; origin xyz=0.031531 -0.0054572 0 rpy=0 0 0 -> xyz=0.031474 -0.0057806 0 rpy=0 0.00014037 -0.020997
- joint R_ring_proximal_joint: limit lower=-1.57 upper=0 effort=10 velocity=0.8 -> lower=-1.602 upper=0 effort=0 velocity=0; origin xyz=-0.009965 0.012307 -0.097841 rpy=0 1.5184 3.1416 -> xyz=-0.0099658 0.0123 -0.095888 rpy=0 1.5184 3.1416
- joint R_ring_tip_joint: origin xyz=0.038 -0.0015 0 rpy=0 0 0 -> xyz=0.0385 -0.0015 0 rpy=0 0 0
- joint R_thumb_distal_joint: limit lower=0 upper=1.23 effort=10 velocity=0.8 -> lower=0 upper=1.267 effort=0 velocity=0; mimic joint=R_thumb_proximal_pitch_joint multiplier=0.974 offset=0 -> joint=R_thumb_proximal_pitch_joint multiplier=1.06 offset=0; origin xyz=0.061444 0.0082822 0 rpy=0 0 1.221E-05 -> xyz=0.061549 0.007464 0 rpy=0 1.7448E-05 -0.055652; parent R_thumb_proximal_link -> R_thumb_proximal_pitch_link
- joint R_thumb_proximal_pitch_joint: child R_thumb_proximal_link -> R_thumb_proximal_pitch_link; limit lower=0 upper=1.22 effort=10 velocity=0.8 -> lower=0 upper=1.159 effort=0 velocity=0; origin xyz=0.02175 0 0 rpy=1.5709 1.221E-05 0 -> xyz=0.02175 -7.414E-05 0 rpy=1.5708 0 -0.0057076; parent R_thumb_proximal_base_link -> R_thumb_proximal_yaw_link
- joint R_thumb_proximal_yaw_joint: child R_thumb_proximal_base_link -> R_thumb_proximal_yaw_link; limit lower=-1.74 upper=0 effort=10 velocity=0.8 -> lower=-1.676 upper=0 effort=0 velocity=0; origin xyz=0.021995 0.015502 -0.024995 rpy=3.1416 0 0 -> xyz=0.022 0.0155 -0.022892 rpy=3.1416 0 0
- joint R_thumb_tip_joint: origin xyz=0.031 0 0 rpy=0 0 0 -> xyz=0.030 -0.0015 0 rpy=0 0 0
